Commit message: Updated rover_arm_mode.urdf with 4 legs and wheels, chassie, antenna. Version 0.1

File: ros/src/rover_world/urdf/rover_arm_mode.urdf (robot description, URDF)
Before this commit: robot rover, 5 links, 4 joints
Links:
- added link Leg_FL, mass 1; collision box size=0.3048 0.127 0.1143; visual box size=0.3048 0.127 0.1143
- added link Leg_FR, mass 1; collision box size=0.3048 0.127 0.1143; visual box size=0.3048 0.127 0.1143
- added link Leg_RL, mass 1; collision box size=0.3048 0.127 0.1143; visual box size=0.3048 0.127 0.1143
- added link Leg_RR, mass 1; collision box size=0.3048 0.127 0.1143; visual box size=0.3048 0.127 0.1143
- added link antenna_link, mass 1; collision cylinder length=1.5748 radius=0.0635; visual cylinder length=1.5748 radius=0.0635
- link Wheel_FL: geometry collision cylinder length=0.254 radius=0.508; visual cylinder length=0.254 radius=0.508
- link Wheel_FR: geometry collision cylinder length=0.254 radius=0.508; visual cylinder length=0.254 radius=0.508
- link Wheel_RL: geometry collision cylinder length=0.254 radius=0.508; visual cylinder length=0.254 radius=0.508
- link Wheel_RR: geometry collision cylinder length=0.254 radius=0.508; visual cylinder length=0.254 radius=0.508
- link base_link: geometry collision box size=1.1176 0.4064 0.127; visual box size=1.1176 0.4064 0.127
Joints:
- added joint Chassie_Leg_FL_Joint: type continuous, parent base_link, child Leg_FL, origin xyz=0 0 0.096 rpy=0 0 0, axis 1 0 0, limit lower=0 upper=0 effort=10.0 velocity=8.94
- added joint Chassie_Leg_FR_Joint: type continuous, parent base_link, child Leg_FR, origin xyz=0 0 0.096 rpy=0 0 0, axis 1 0 0, limit lower=0 upper=0 effort=10.0 velocity=8.94
- added joint Chassie_Leg_RL_Joint: type continuous, parent base_link, child Leg_RL, origin xyz=0 0 0.096 rpy=0 0 0, axis 1 0 0, limit lower=0 upper=0 effort=10.0 velocity=8.94
- added joint Chassie_Leg_RR_Joint: type continuous, parent base_link, child Leg_RR, origin xyz=0 0 0.096 rpy=0 0 0, axis 1 0 0, limit lower=0 upper=0 effort=10.0 velocity=8.94
- added joint Chassie_antenna_link_Joint: type continuous, parent base_link, child antenna_link, origin xyz=0 0 0.096 rpy=0 0 0, axis 1 0 0, limit lower=0 upper=0 effort=10.0 velocity=8.94
- joint Chassie_Wheel_FL_Joint: parent base_link -> Leg_FL
- joint Chassie_Wheel_FR_Joint: parent base_link -> Leg_FR
- joint Chassie_Wheel_RL_Joint: parent base_link -> Leg_RL
- joint Chassie_Wheel_RR_Joint: parent base_link -> Leg_RR
