Commit message: Reposition left and right ZED camera lenses

File: ros/src/rover_world/sim_world/models/auto_mode/auto_mode.xacro (robot description, xacro)
@@ -3,9 +3,9 @@
 <robot name="auto_mode" xmlns:xacro="http://www.ros.org/wiki/xacro">
   <!-- Start by including all required xacro files which hold the macros -->
+  <xacro:include filename="$(find sim_world)/models/common_models/common_models.xacro" />
   <xacro:include filename="$(find sim_world)/models/auto_mode/auto_mode.gazebo" />
   <xacro:include filename="$(find sim_world)/models/auto_mode/materials.xacro" />
   <xacro:include filename="$(find sim_world)/models/auto_mode/macros.xacro"    />
   <xacro:include filename="$(find sim_world)/models/auto_mode/parameter.xacro" />
-  <xacro:include filename="$(find sim_world)/models/common_models/common_models.xacro" />
   <!-- Add the ZED camera -->
   <link name="zed_cam_link">
@@ -15,5 +15,5 @@
     </inertial>
     <collision name="collision">
-      <origin xyz="${x_chassis/2} 0 ${(z_chassis/2)+z_zed_cam}" rpy="0 0 ${pi/2}"/>
+      <origin xyz="${x_pose_zed_cam} 0 ${z_pose_zed_cam}" rpy="0 0 ${pi/2}"/>
       <geometry>
         <box size="${x_zed_cam} ${y_zed_cam} ${z_zed_cam}"/>
@@ -21,5 +21,5 @@
     </collision>
     <visual name="zed_cam_visual">
-      <origin xyz="${x_chassis/2} 0 ${(z_chassis/2)+z_zed_cam}" rpy="0 0 ${pi/2}"/>
+      <origin xyz="${x_pose_zed_cam} 0 ${z_pose_zed_cam}" rpy="0 0 ${pi/2}"/>
       <geometry>
         <box size="${x_zed_cam} ${y_zed_cam} ${z_zed_cam}"/>

File: ros/src/rover_world/sim_world/models/auto_mode/parameter.xacro (robot description, xacro)
@@ -2,5 +2,10 @@
 <robot xmlns:xacro="http://www.ros.org/wiki/xacro">
   <!-- Define parameter for the autonomous subsystem -->
+  <!-- TODO: Apart from separation, all values need to be changed from ZED cam to ZED mini -->
   <!-- Parameters for ZED camera. See: https://www.stereolabs.com/zed/ -->
+  <!-- Origin (these values are temporary until I find out more about how it's mounted) -->
+  <xacro:property name="x_pose_zed_cam" value="${x_chassis/2}" />
+  <xacro:property name="y_pose_zed_cam" value="0" />
+  <xacro:property name="z_pose_zed_cam" value="${(z_chassis/2)+z_zed_cam}" />
   <!-- Physical parameters: xyz [m] and mass [kg] -->
   <xacro:property name="x_zed_cam" value="0.175" />
@@ -25,3 +30,5 @@
   <xacro:property name="dep_min_zed_cam" value="0.3" />
   <xacro:property name="dep_max_zed_cam" value="25.0" />
+  <!-- separation between left and right sensors -->
+  <xacro:property name="l_r_sep_zed_cam" value="0.063" />
 </robot>
