Commit message: Updated common_models.xarco, added the antenna onto the chassis. Controlling is still an issue.

File: ros/src/rover_world/sim_world/models/common_models/common_models.xacro (robot description, xacro)
@@ -60,6 +60,19 @@
       </geometry>
     </visual> -->
-  </link>
-  <!-- Test Leg -->
+    <!-- Add antenna to the rover -->
+    <collision name="antenna">
+      <origin xyz="${-x_chassis/2-r_antenna} 0 ${l_antenna/2-z_chassis/2}" rpy="0 0 0"/>
+      <geometry>
+        <cylinder radius="${r_antenna}" length="${l_antenna}"/>
+      </geometry>
+    </collision>
+    <visual name="antenna_visual">
+      <origin xyz="${-x_chassis/2-r_antenna} 0 ${l_antenna/2-z_chassis/2}" rpy="0 0 0"/>
+      <geometry>
+        <cylinder radius="${r_antenna}" length="${l_antenna}"/>
+      </geometry>
+    </visual>
+  </link>
+  <!-- Add legs for the robot -->
   <link name="leg_rl">
     <inertial>
@@ -195,5 +208,4 @@
     </inertial>
   </link>
-  <!--TEST-->
   <link name="wheel_fr">
     <collision name="collision">

Commit message: Changed explicit 1.5707 to precise 90 degs

File: ros/src/rover_world/sim_world/models/common_models/common_models.xacro (robot description, xacro)
@@ -81,5 +81,5 @@
     </inertial>
     <collision name="collision">
-      <origin xyz="0 0 0" rpy="0 0 1.5707"/>
+      <origin xyz="0 0 0" rpy="0 0 ${pi/2}"/>
       <geometry>
         <box size="${l_leg} ${w_leg} ${h_leg}"/>
@@ -87,5 +87,5 @@
     </collision>
     <visual name="leg_rl_visual">
-      <origin xyz="0 0 0" rpy="0 0 1.5707"/>
+      <origin xyz="0 0 0" rpy="0 0 ${pi/2}"/>
       <geometry>
         <box size="${l_leg} ${w_leg} ${h_leg}"/>
@@ -99,5 +99,5 @@
     </inertial>
     <collision name="collision">
-      <origin xyz="0 0 0" rpy="0 0 1.5707"/>
+      <origin xyz="0 0 0" rpy="0 0 ${pi/2}"/>
       <geometry>
         <box size="${l_leg} ${w_leg} ${h_leg}"/>
@@ -105,5 +105,5 @@
     </collision>
     <visual name="leg_rr_visual">
-      <origin xyz="0 0 0" rpy="0 0 1.5707"/>
+      <origin xyz="0 0 0" rpy="0 0 ${pi/2}"/>
       <geometry>
         <box size="${l_leg} ${w_leg} ${h_leg}"/>
@@ -117,5 +117,5 @@
     </inertial>
     <collision name="collision">
-      <origin xyz="0 0 0" rpy="0 0 1.5707"/>
+      <origin xyz="0 0 0" rpy="0 0 ${pi/2}"/>
       <geometry>
         <box size="${l_leg} ${w_leg} ${h_leg}"/>
@@ -123,5 +123,5 @@
     </collision>
     <visual name="leg_fl_visual">
-      <origin xyz="0 0 0" rpy="0 0 1.5707"/>
+      <origin xyz="0 0 0" rpy="0 0 ${pi/2}"/>
       <geometry>
         <box size="${l_leg} ${w_leg} ${h_leg}"/>
@@ -135,5 +135,5 @@
     </inertial>
     <collision name="collision">
-      <origin xyz="0 0 0" rpy="0 0 1.5707"/>
+      <origin xyz="0 0 0" rpy="0 0 ${pi/2}"/>
       <geometry>
         <box size="${l_leg} ${w_leg} ${h_leg}"/>
@@ -141,5 +141,5 @@
     </collision>
     <visual name="leg_fr_visual">
-      <origin xyz="0 0 0" rpy="0 0 1.5707"/>
+      <origin xyz="0 0 0" rpy="0 0 ${pi/2}"/>
       <geometry>
         <box size="${l_leg} ${w_leg} ${h_leg}"/>
@@ -150,5 +150,5 @@
   <link name="wheel_rl">
     <collision name="collision">
-      <origin xyz="0 0 0" rpy="0 1.5707 1.5707"/>
+      <origin xyz="0 0 0" rpy="0 ${pi/2} ${pi/2}"/>
       <geometry>
         <cylinder radius="${r_wheel}" length="${h_wheel}"/>
@@ -166,11 +166,11 @@
     </collision>
     <visual name="wheel_rl_visual">
-      <origin xyz="0 0 0" rpy="0 1.5707 1.5707"/>
-      <geometry>
-        <cylinder radius="${r_wheel}" length="${h_wheel}"/>
-      </geometry>
-    </visual>
-    <inertial>
-      <origin xyz="0 0 0" rpy="0 1.5707 1.5707"/>
+      <origin xyz="0 0 0" rpy="0 ${pi/2} ${pi/2}"/>
+      <geometry>
+        <cylinder radius="${r_wheel}" length="${h_wheel}"/>
+      </geometry>
+    </visual>
+    <inertial>
+      <origin xyz="0 0 0" rpy="0 ${pi/2} ${pi/2}"/>
       <mass value="${m_wheel}"/>
       <cylinder_inertia m="${m_wheel}" r="${r_wheel}" h="${h_wheel}"/>
@@ -180,5 +180,5 @@
   <link name="wheel_rr">
     <collision name="collision">
-      <origin xyz="0 0 0" rpy="0 1.5707 1.5707"/>
+      <origin xyz="0 0 0" rpy="0 ${pi/2} ${pi/2}"/>
       <geometry>
         <cylinder radius="${r_wheel}" length="${h_wheel}"/>
@@ -196,11 +196,11 @@
     </collision>
     <visual name="wheel_rr_visual">
-      <origin xyz="0 0 0" rpy="0 1.5707 1.5707"/>
-      <geometry>
-        <cylinder radius="${r_wheel}" length="${h_wheel}"/>
-      </geometry>
-    </visual>
-    <inertial>
-      <origin xyz="0 0 0" rpy="0 1.5707 1.5707"/>
+      <origin xyz="0 0 0" rpy="0 ${pi/2} ${pi/2}"/>
+      <geometry>
+        <cylinder radius="${r_wheel}" length="${h_wheel}"/>
+      </geometry>
+    </visual>
+    <inertial>
+      <origin xyz="0 0 0" rpy="0 ${pi/2} ${pi/2}"/>
       <mass value="${m_wheel}"/>
       <cylinder_inertia m="${m_wheel}" r="${r_wheel}" h="${h_wheel}"/>
@@ -210,5 +210,5 @@
   <link name="wheel_fr">
     <collision name="collision">
-      <origin xyz="0 0 0" rpy="0 1.5707 1.5707"/>
+      <origin xyz="0 0 0" rpy="0 ${pi/2} ${pi/2}"/>
       <geometry>
         <cylinder radius="${r_wheel}" length="${h_wheel}"/>
@@ -226,11 +226,11 @@
     </collision>
     <visual name="wheel_fr_visual">
-      <origin xyz="0 0 0" rpy="0 1.5707 1.5707"/>
-      <geometry>
-        <cylinder radius="${r_wheel}" length="${h_wheel}"/>
-      </geometry>
-    </visual>
-    <inertial>
-      <origin xyz="0 0 0" rpy="0 1.5707 1.5707"/>
+      <origin xyz="0 0 0" rpy="0 ${pi/2} ${pi/2}"/>
+      <geometry>
+        <cylinder radius="${r_wheel}" length="${h_wheel}"/>
+      </geometry>
+    </visual>
+    <inertial>
+      <origin xyz="0 0 0" rpy="0 ${pi/2} ${pi/2}"/>
       <mass value="${m_wheel}"/>
       <cylinder_inertia m="${m_wheel}" r="${r_wheel}" h="${h_wheel}"/>
@@ -240,5 +240,5 @@
   <link name="wheel_fl">
     <collision name="collision">
-      <origin xyz="0 0 0" rpy="0 1.5707 1.5707"/>
+      <origin xyz="0 0 0" rpy="0 ${pi/2} ${pi/2}"/>
       <geometry>
         <cylinder radius="${r_wheel}" length="${h_wheel}"/>
@@ -256,11 +256,11 @@
     </collision>
     <visual name="wheel_fl_visual">
-      <origin xyz="0 0 0" rpy="0 1.5707 1.5707"/>
-      <geometry>
-        <cylinder radius="${r_wheel}" length="${h_wheel}"/>
-      </geometry>
-    </visual>
-    <inertial>
-      <origin xyz="0 0 0" rpy="0 1.5707 1.5707"/>
+      <origin xyz="0 0 0" rpy="0 ${pi/2} ${pi/2}"/>
+      <geometry>
+        <cylinder radius="${r_wheel}" length="${h_wheel}"/>
+      </geometry>
+    </visual>
+    <inertial>
+      <origin xyz="0 0 0" rpy="0 ${pi/2} ${pi/2}"/>
       <mass value="${m_wheel}"/>
       <cylinder_inertia m="${m_wheel}" r="${r_wheel}" h="${h_wheel}"/>

Commit message: Fix bug where rover was not subscribing to cmd_vel

File: ros/src/rover_world/sim_world/models/common_models/common_models.xacro (robot description, xacro)
@@ -270,5 +270,5 @@
   <!-- Set joints for the wheels which can be controlled over ROS -->
   <!-- it is continuous since it is a wheel-->
-  <joint type="continuous" name="leg_fr_joint_wheel_rl">
+  <joint type="continuous" name="leg_rl_joint_wheel_rl">
     <origin xyz="0 ${l_leg/2+h_wheel/2} ${r_wheel/2-z_chassis/2}" rpy="0 0 0"/>
     <child link="wheel_rl"/>
