Commit message: Updated with four wheels that work with controls

File: ros/src/rover_world/sim_world/models/arm_mode/arm_mode.xacro (robot description, xacro)
@@ -62,52 +62,114 @@
   </link>
   <!-- Add the wheels for the robot -->
-  <link name="left_wheel">
-    <collision name="collision">
-      <origin xyz="0 0 0" rpy="0 1.5707 1.5707"/>
-      <geometry>
-        <cylinder radius="${r_wheel}" length="${h_wheel}"/>
-      </geometry>
-      <surface>
-        <friction>
-          <ode>
-            <mu>1.0</mu>
-            <mu2>1.0</mu2>
-            <slip1>0.0</slip1>
-            <slip2>0.0</slip2>
-          </ode>
-        </friction>
-      </surface>
-    </collision>
-    <visual name="left_wheel_visual">
-      <origin xyz="0 0 0" rpy="0 1.5707 1.5707"/>
-      <geometry>
-        <cylinder radius="${r_wheel}" length="${h_wheel}"/>
-      </geometry>
-    </visual>
-    <inertial>
-      <origin xyz="0 0 0" rpy="0 1.5707 1.5707"/>
-      <mass value="${m_wheel}"/>
-      <cylinder_inertia m="${m_wheel}" r="${r_wheel}" h="${h_wheel}"/>
-      <xacro:cylinder_inertia m="${m_wheel}" r="${r_wheel}" h="${h_wheel}"/>
-    </inertial>
-  </link>
-  <link name="right_wheel">
-    <collision name="collision">
-      <origin xyz="0 0 0" rpy="0 1.5707 1.5707"/>
-      <geometry>
-        <cylinder radius="${r_wheel}" length="${h_wheel}"/>
-      </geometry>
-      <surface>
-        <friction>
-          <ode>
-            <mu>1.0</mu>
-            <mu2>1.0</mu2>
-            <slip1>0.0</slip1>
-            <slip2>0.0</slip2>
-          </ode>
-        </friction>
-      </surface>
-    </collision>
-    <visual name="right_wheel_visual">
+  <link name="wheel_rl">
+    <collision name="collision">
+      <origin xyz="0 0 0" rpy="0 1.5707 1.5707"/>
+      <geometry>
+        <cylinder radius="${r_wheel}" length="${h_wheel}"/>
+      </geometry>
+      <surface>
+        <friction>
+          <ode>
+            <mu>1.0</mu>
+            <mu2>1.0</mu2>
+            <slip1>0.0</slip1>
+            <slip2>0.0</slip2>
+          </ode>
+        </friction>
+      </surface>
+    </collision>
+    <visual name="wheel_rl_visual">
+      <origin xyz="0 0 0" rpy="0 1.5707 1.5707"/>
+      <geometry>
+        <cylinder radius="${r_wheel}" length="${h_wheel}"/>
+      </geometry>
+    </visual>
+    <inertial>
+      <origin xyz="0 0 0" rpy="0 1.5707 1.5707"/>
+      <mass value="${m_wheel}"/>
+      <cylinder_inertia m="${m_wheel}" r="${r_wheel}" h="${h_wheel}"/>
+      <xacro:cylinder_inertia m="${m_wheel}" r="${r_wheel}" h="${h_wheel}"/>
+    </inertial>
+  </link>
+  <link name="wheel_rr">
+    <collision name="collision">
+      <origin xyz="0 0 0" rpy="0 1.5707 1.5707"/>
+      <geometry>
+        <cylinder radius="${r_wheel}" length="${h_wheel}"/>
+      </geometry>
+      <surface>
+        <friction>
+          <ode>
+            <mu>1.0</mu>
+            <mu2>1.0</mu2>
+            <slip1>0.0</slip1>
+            <slip2>0.0</slip2>
+          </ode>
+        </friction>
+      </surface>
+    </collision>
+    <visual name="wheel_rr_visual">
+      <origin xyz="0 0 0" rpy="0 1.5707 1.5707"/>
+      <geometry>
+        <cylinder radius="${r_wheel}" length="${h_wheel}"/>
+      </geometry>
+    </visual>
+    <inertial>
+      <origin xyz="0 0 0" rpy="0 1.5707 1.5707"/>
+      <mass value="${m_wheel}"/>
+      <cylinder_inertia m="${m_wheel}" r="${r_wheel}" h="${h_wheel}"/>
+      <xacro:cylinder_inertia m="${m_wheel}" r="${r_wheel}" h="${h_wheel}"/>
+    </inertial>
+  </link>
+  <!--TEST-->
+  <link name="wheel_fr">
+    <collision name="collision">
+      <origin xyz="0 0 0" rpy="0 1.5707 1.5707"/>
+      <geometry>
+        <cylinder radius="${r_wheel}" length="${h_wheel}"/>
+      </geometry>
+      <surface>
+        <friction>
+          <ode>
+            <mu>1.0</mu>
+            <mu2>1.0</mu2>
+            <slip1>0.0</slip1>
+            <slip2>0.0</slip2>
+          </ode>
+        </friction>
+      </surface>
+    </collision>
+    <visual name="wheel_fr_visual">
+      <origin xyz="0 0 0" rpy="0 1.5707 1.5707"/>
+      <geometry>
+        <cylinder radius="${r_wheel}" length="${h_wheel}"/>
+      </geometry>
+    </visual>
+    <inertial>
+      <origin xyz="0 0 0" rpy="0 1.5707 1.5707"/>
+      <mass value="${m_wheel}"/>
+      <cylinder_inertia m="${m_wheel}" r="${r_wheel}" h="${h_wheel}"/>
+      <xacro:cylinder_inertia m="${m_wheel}" r="${r_wheel}" h="${h_wheel}"/>
+    </inertial>
+  </link>
+  <!--TEST-->
+  <link name="wheel_fl">
+    <collision name="collision">
+      <origin xyz="0 0 0" rpy="0 1.5707 1.5707"/>
+      <geometry>
+        <cylinder radius="${r_wheel}" length="${h_wheel}"/>
+      </geometry>
+      <surface>
+        <friction>
+          <ode>
+            <mu>1.0</mu>
+            <mu2>1.0</mu2>
+            <slip1>0.0</slip1>
+            <slip2>0.0</slip2>
+          </ode>
+        </friction>
+      </surface>
+    </collision>
+    <visual name="wheel_fl_visual">
       <origin xyz="0 0 0" rpy="0 1.5707 1.5707"/>
       <geometry>
@@ -124,7 +186,7 @@
   <!-- Set joints for the wheels which can be controlled over ROS -->
   <!-- it is continuous since it is a wheel-->
-  <joint type="continuous" name="left_wheel_hinge">
+  <joint type="continuous" name="base_link_joint_wheel_rl">
     <origin xyz="${-x_chassis/4} ${y_chassis/2+h_wheel/2} ${r_wheel/2-z_chassis/2}" rpy="0 0 0"/>
-    <child link="left_wheel"/>
+    <child link="wheel_rl"/>
     <parent link="base_link"/>
     <axis xyz="0 1 0" rpy="0 0 0"/>
@@ -133,7 +195,24 @@
     <joint_properties damping="0.0" friction="0.0"/>
   </joint>
-  <joint type="continuous" name="right_wheel_hinge">
+  <joint type="continuous" name="base_link_joint_wheel_rr">
     <origin xyz="${-x_chassis/4} ${-y_chassis/2-h_wheel/2} ${r_wheel/2-z_chassis/2}" rpy="0 0 0"/>
-    <child link="right_wheel"/>
+    <child link="wheel_rr"/>
+    <parent link="base_link"/>
+    <axis xyz="0 1 0" rpy="0 0 0"/>
+    <limit effort="100" velocity="100"/>
+    <joint_properties damping="0.0" friction="0.0"/>
+  </joint>
+  <!--TEST-->
+  <joint type="continuous" name="base_link_joint_wheel_fr">
+    <origin xyz="${x_chassis/4} ${-y_chassis/2-h_wheel/2} ${r_wheel/2-z_chassis/2}" rpy="0 0 0"/>
+    <child link="wheel_fr"/>
+    <parent link="base_link"/>
+    <axis xyz="0 1 0" rpy="0 0 0"/>
+    <limit effort="100" velocity="100"/>
+    <joint_properties damping="0.0" friction="0.0"/>
+  </joint>
+    <joint type="continuous" name="base_link_joint_wheel_fl">
+    <origin xyz="${x_chassis/4} ${y_chassis/2+h_wheel/2} ${r_wheel/2-z_chassis/2}" rpy="0 0 0"/>
+    <child link="wheel_fl"/>
     <parent link="base_link"/>
     <axis xyz="0 1 0" rpy="0 0 0"/>

File: ros/src/rover_world/sim_world/models/arm_mode/parameter.xacro (robot description, xacro)
@@ -13,3 +13,10 @@
   <xacro:property name="torque_wheel" value="10" />
   <xacro:property name="L_wheel" value="0.1788" />
+  <!-- Parameter for the legs, length [m], width [m], height [m]-->
+  <xacro:property name="l_leg" value="0.3048" />
+  <xacro:property name="w_leg" value="0.127" />
+  <xacro:property name="h_leg" value="0.1143" />
+  <!-- Parameter for the antenna, radius [m], length [m] -->
+  <xacro:property name="r_antenna" value="0.0635" />
+  <xacro:property name="l_antenna" value="1.5748" />
 </robot>

Commit message: Updated arm_mode.xarco and paramete.xarco with the correct dimesions of the rover for the wheels and the cassis.

File: ros/src/rover_world/sim_world/models/arm_mode/arm_mode.xacro (robot description, xacro)
@@ -38,5 +38,5 @@
     </visual>
     <!-- Add the caster wheel! Here we simply assume complete slippage, thus we do not require that it rotates! -->
-    <collision name='caster_collision'>
+    <!-- <collision name='caster_collision'>
       <origin xyz="${-(r_wheel/2)+x_chassis/2} 0 ${-z_chassis/2}" rpy=" 0 0 0"/>
       <geometry>
@@ -59,5 +59,5 @@
         <sphere radius="${r_wheel/2}"/>
       </geometry>
-    </visual>
+    </visual> -->
   </link>
   <!-- Add the wheels for the robot -->
@@ -187,5 +187,5 @@
   <!-- it is continuous since it is a wheel-->
   <joint type="continuous" name="base_link_joint_wheel_rl">
-    <origin xyz="${-x_chassis/4} ${y_chassis/2+h_wheel/2} ${r_wheel/2-z_chassis/2}" rpy="0 0 0"/>
+    <origin xyz="${-wheel_dist_center} ${y_chassis/2+h_wheel/2} ${r_wheel/2-z_chassis/2}" rpy="0 0 0"/>
     <child link="wheel_rl"/>
     <parent link="base_link"/>
@@ -196,5 +196,5 @@
   </joint>
   <joint type="continuous" name="base_link_joint_wheel_rr">
-    <origin xyz="${-x_chassis/4} ${-y_chassis/2-h_wheel/2} ${r_wheel/2-z_chassis/2}" rpy="0 0 0"/>
+    <origin xyz="${-wheel_dist_center} ${-y_chassis/2-h_wheel/2} ${r_wheel/2-z_chassis/2}" rpy="0 0 0"/>
     <child link="wheel_rr"/>
     <parent link="base_link"/>
@@ -205,5 +205,5 @@
   <!--TEST-->
   <joint type="continuous" name="base_link_joint_wheel_fr">
-    <origin xyz="${x_chassis/4} ${-y_chassis/2-h_wheel/2} ${r_wheel/2-z_chassis/2}" rpy="0 0 0"/>
+    <origin xyz="${wheel_dist_center} ${-y_chassis/2-h_wheel/2} ${r_wheel/2-z_chassis/2}" rpy="0 0 0"/>
     <child link="wheel_fr"/>
     <parent link="base_link"/>
@@ -213,5 +213,5 @@
   </joint>
     <joint type="continuous" name="base_link_joint_wheel_fl">
-    <origin xyz="${x_chassis/4} ${y_chassis/2+h_wheel/2} ${r_wheel/2-z_chassis/2}" rpy="0 0 0"/>
+    <origin xyz="${wheel_dist_center} ${y_chassis/2+h_wheel/2} ${r_wheel/2-z_chassis/2}" rpy="0 0 0"/>
     <child link="wheel_fl"/>
     <parent link="base_link"/>

File: ros/src/rover_world/sim_world/models/arm_mode/parameter.xacro (robot description, xacro)
@@ -3,14 +3,15 @@
   <!-- Define parameter for the differential drive robot -->
   <!-- Parameter for the chassis, size [m] and mass [kg] -->
-  <xacro:property name="x_chassis" value="0.5" />
-  <xacro:property name="y_chassis" value="0.3" />
-  <xacro:property name="z_chassis" value="0.15" />
+  <xacro:property name="x_chassis" value="1.1176" />
+  <xacro:property name="y_chassis" value="0.4064" />
+  <xacro:property name="z_chassis" value="0.127" />
   <xacro:property name="m_chassis" value="10.0" />
   <!-- Parameter for the wheels, radius [m], height [m], mass [kg], torque [Nm], wheelbase [m] -->
-  <xacro:property name="r_wheel" value="0.1075"/>
-  <xacro:property name="h_wheel" value="0.03" />
+  <xacro:property name="r_wheel" value="0.254"/>
+  <xacro:property name="h_wheel" value="0.254" />
   <xacro:property name="m_wheel" value="3.0" />
   <xacro:property name="torque_wheel" value="10" />
   <xacro:property name="L_wheel" value="0.1788" />
+  <xacro:property name="wheel_dist_center" value="0.5588" />
   <!-- Parameter for the legs, length [m], width [m], height [m]-->
   <xacro:property name="l_leg" value="0.3048" />

Commit message: Updated arm_mode.xacro, arm_mode.gazebo, and parameters.xarco with leg links and joints between wheels-legs-chassis. Keyboard controls are not working due to either odom-cmd/topic not activated.

File: ros/src/rover_world/sim_world/models/arm_mode/arm_mode.xacro (robot description, xacro)
@@ -61,4 +61,77 @@
     </visual> -->
   </link>
+  <!-- Test Leg -->
+  <link name="leg_rl">
+    <inertial>
+      <mass value="${m_leg}"/>
+      <xacro:box_inertia m="${m_leg}" x="${l_leg}" y="${w_leg}" z="${h_leg}"/>
+    </inertial>
+    <collision name="collision">
+      <origin xyz="0 0 0" rpy="0 0 1.5707"/>
+      <geometry>
+        <box size="${l_leg} ${w_leg} ${h_leg}"/>
+      </geometry>
+    </collision>
+    <visual name="leg_rl_visual">
+      <origin xyz="0 0 0" rpy="0 0 1.5707"/>
+      <geometry>
+        <box size="${l_leg} ${w_leg} ${h_leg}"/>
+      </geometry>
+    </visual>
+  </link>
+  <link name="leg_rr">
+    <inertial>
+      <mass value="${m_leg}"/>
+      <xacro:box_inertia m="${m_leg}" x="${l_leg}" y="${w_leg}" z="${h_leg}"/>
+    </inertial>
+    <collision name="collision">
+      <origin xyz="0 0 0" rpy="0 0 1.5707"/>
+      <geometry>
+        <box size="${l_leg} ${w_leg} ${h_leg}"/>
+      </geometry>
+    </collision>
+    <visual name="leg_rr_visual">
+      <origin xyz="0 0 0" rpy="0 0 1.5707"/>
+      <geometry>
+        <box size="${l_leg} ${w_leg} ${h_leg}"/>
+      </geometry>
+    </visual>
+  </link>
+  <link name="leg_fl">
+    <inertial>
+      <mass value="${m_leg}"/>
+      <xacro:box_inertia m="${m_leg}" x="${l_leg}" y="${w_leg}" z="${h_leg}"/>
+    </inertial>
+    <collision name="collision">
+      <origin xyz="0 0 0" rpy="0 0 1.5707"/>
+      <geometry>
+        <box size="${l_leg} ${w_leg} ${h_leg}"/>
+      </geometry>
+    </collision>
+    <visual name="leg_fl_visual">
+      <origin xyz="0 0 0" rpy="0 0 1.5707"/>
+      <geometry>
+        <box size="${l_leg} ${w_leg} ${h_leg}"/>
+      </geometry>
+    </visual>
+  </link>
+  <link name="leg_fr">
+    <inertial>
+      <mass value="${m_leg}"/>
+      <xacro:box_inertia m="${m_leg}" x="${l_leg}" y="${w_leg}" z="${h_leg}"/>
+    </inertial>
+    <collision name="collision">
+      <origin xyz="0 0 0" rpy="0 0 1.5707"/>
+      <geometry>
+        <box size="${l_leg} ${w_leg} ${h_leg}"/>
+      </geometry>
+    </collision>
+    <visual name="leg_fr_visual">
+      <origin xyz="0 0 0" rpy="0 0 1.5707"/>
+      <geometry>
+        <box size="${l_leg} ${w_leg} ${h_leg}"/>
+      </geometry>
+    </visual>
+  </link>
   <!-- Add the wheels for the robot -->
   <link name="wheel_rl">
@@ -153,5 +226,4 @@
     </inertial>
   </link>
-  <!--TEST-->
   <link name="wheel_fl">
     <collision name="collision">
@@ -186,34 +258,65 @@
   <!-- Set joints for the wheels which can be controlled over ROS -->
   <!-- it is continuous since it is a wheel-->
-  <joint type="continuous" name="base_link_joint_wheel_rl">
+  <joint type="continuous" name="leg_fr_joint_wheel_rl">
+    <origin xyz="0 ${l_leg/2+h_wheel/2} ${r_wheel/2-z_chassis/2}" rpy="0 0 0"/>
+    <child link="wheel_rl"/>
+    <parent link="leg_rl"/>
+    <axis xyz="0 1 0" rpy="0 0 0"/>
+    <!-- velocity here is the max allowed velocity not the acutal velocity-->
+    <limit effort="100" velocity="100"/>
+    <joint_properties damping="0.0" friction="0.0"/>
+  </joint>
+  <joint type="continuous" name="leg_rr_joint_wheel_rr">
+    <origin xyz="0 ${-y_chassis/2-h_wheel/2} ${r_wheel/2-z_chassis/2}" rpy="0 0 0"/>
+    <child link="wheel_rr"/>
+    <parent link="leg_rr"/>
+    <axis xyz="0 1 0" rpy="0 0 0"/>
+    <limit effort="100" velocity="100"/>
+    <joint_properties damping="0.0" friction="0.0"/>
+  </joint>
+  <joint type="continuous" name="leg_fr_joint_wheel_fr">
+    <origin xyz="0 ${-l_leg/2-h_wheel/2} ${r_wheel/2-z_chassis/2}" rpy="0 0 0"/>
+    <child link="wheel_fr"/>
+    <parent link="leg_fr"/>
+    <axis xyz="0 1 0" rpy="0 0 0"/>
+    <limit effort="100" velocity="100"/>
+    <joint_properties damping="0.0" friction="0.0"/>
+  </joint>
+  <joint type="continuous" name="leg_fl_joint_wheel_fl">
+    <origin xyz="0 ${l_leg/2+h_wheel/2} ${r_wheel/2-z_chassis/2}" rpy="0 0 0"/>
+    <child link="wheel_fl"/>
+    <parent link="leg_fl"/>
+    <axis xyz="0 1 0" rpy="0 0 0"/>
+    <limit effort="100" velocity="100"/>
+    <joint_properties damping="0.0" friction="0.0"/>
+  </joint>
+   <joint type="revolute" name="chassis_link_joint_leg_rl">
     <origin xyz="${-wheel_dist_center} ${y_chassis/2+h_wheel/2} ${r_wheel/2-z_chassis/2}" rpy="0 0 0"/>
-    <child link="wheel_rl"/>
-    <parent link="base_link"/>
-    <axis xyz="0 1 0" rpy="0 0 0"/>
-    <!-- velocity here is the max allowed velocity not the acutal velocity-->
-    <limit effort="100" velocity="100"/>
-    <joint_properties damping="0.0" friction="0.0"/>
-  </joint>
-  <joint type="continuous" name="base_link_joint_wheel_rr">
+    <child link="leg_rl"/>
+    <parent link="chassis_link"/>
+    <axis xyz="0 1 0" rpy="0 0 0"/>
+    <limit effort="100" velocity="100"/>
+    <joint_properties damping="0.0" friction="0.0"/>
+  </joint>
+  <joint type="revolute" name="chassis_link_joint_leg_rr">
     <origin xyz="${-wheel_dist_center} ${-y_chassis/2-h_wheel/2} ${r_wheel/2-z_chassis/2}" rpy="0 0 0"/>
-    <child link="wheel_rr"/>
-    <parent link="base_link"/>
-    <axis xyz="0 1 0" rpy="0 0 0"/>
-    <limit effort="100" velocity="100"/>
-    <joint_properties damping="0.0" friction="0.0"/>
-  </joint>
-  <!--TEST-->
-  <joint type="continuous" name="base_link_joint_wheel_fr">
+    <child link="leg_rr"/>
+    <parent link="chassis_link"/>
+    <axis xyz="0 1 0" rpy="0 0 0"/>
+    <limit effort="100" velocity="100"/>
+    <joint_properties damping="0.0" friction="0.0"/>
+  </joint>
+  <joint type="revolute" name="chassis_link_joint_leg_fl">
+    <origin xyz="${wheel_dist_center} ${y_chassis/2+h_wheel/2} ${r_wheel/2-z_chassis/2}" rpy="0 0 0"/>
+    <child link="leg_fl"/>
+    <parent link="chassis_link"/>
+    <axis xyz="0 1 0" rpy="0 0 0"/>
+    <limit effort="100" velocity="100"/>
+    <joint_properties damping="0.0" friction="0.0"/>
+  </joint>
+  <joint type="revolute" name="chassis_link_joint_leg_fr">
     <origin xyz="${wheel_dist_center} ${-y_chassis/2-h_wheel/2} ${r_wheel/2-z_chassis/2}" rpy="0 0 0"/>
-    <child link="wheel_fr"/>
-    <parent link="base_link"/>
-    <axis xyz="0 1 0" rpy="0 0 0"/>
-    <limit effort="100" velocity="100"/>
-    <joint_properties damping="0.0" friction="0.0"/>
-  </joint>
-    <joint type="continuous" name="base_link_joint_wheel_fl">
-    <origin xyz="${wheel_dist_center} ${y_chassis/2+h_wheel/2} ${r_wheel/2-z_chassis/2}" rpy="0 0 0"/>
-    <child link="wheel_fl"/>
-    <parent link="base_link"/>
+    <child link="leg_fr"/>
+    <parent link="chassis_link"/>
     <axis xyz="0 1 0" rpy="0 0 0"/>
     <limit effort="100" velocity="100"/>

File: ros/src/rover_world/sim_world/models/arm_mode/parameter.xacro (robot description, xacro)
@@ -14,8 +14,9 @@
   <xacro:property name="L_wheel" value="0.1788" />
   <xacro:property name="wheel_dist_center" value="0.5588" />
-  <!-- Parameter for the legs, length [m], width [m], height [m]-->
+  <!-- Parameter for the legs, length [m], width [m], height [m], mass [kg]-->
   <xacro:property name="l_leg" value="0.3048" />
-  <xacro:property name="w_leg" value="0.127" />
+  <xacro:property name="w_leg" value="0.1270" />
   <xacro:property name="h_leg" value="0.1143" />
+  <xacro:property name="m_leg" value="2.0" />
   <!-- Parameter for the antenna, radius [m], length [m] -->
   <xacro:property name="r_antenna" value="0.0635" />
