Commit message: Added the common_models folder to the models directory. The goal of this was to move the drive train that was located in the arm_mode to the common_models folder so we just need one instance of the drive trian model and then use a one line xarco include to add it to the arm_mode,sci_mode, and auto_mode. The common_models folder can also be used for anything else that will be needed for all 3 configurations.

File: ros/src/rover_world/sim_world/models/arm_mode/arm_mode.xacro (robot description, xacro)
@@ -7,319 +7,4 @@
   <xacro:include filename="$(find sim_world)/models/arm_mode/macros.xacro"    />
   <xacro:include filename="$(find sim_world)/models/arm_mode/parameter.xacro" />
- <!-- Create a dummy link as base link -->
-  <link name='base_link'>
-    <pose>0 0 0 0 0 0</pose>
-  </link>
-  <joint type="fixed" name="base_link_to_chassis">
-    <child link="chassis_link"/>
-    <parent link="base_link"/>
-  </joint>
-  <!-- Define the chassis of the differential drive robot, which is our base -->
-  <link name='chassis_link'>
-    <pose>0 0 0 0 0 0</pose>
-    <!-- Define inertial system for the chassis -->
-    <inertial>
-      <mass value="${m_chassis}"/>
-      <xacro:box_inertia m="${m_chassis}" x="${x_chassis}" y="${y_chassis}" z="${z_chassis}"/>
-    </inertial>
-    <!-- Define collision sorrounding box -->
-    <collision name='collision'>
-      <origin xyz="0 0 0" rpy=" 0 0 0"/>
-      <geometry>
-        <box size="${x_chassis} ${y_chassis} ${z_chassis}"/>
-      </geometry>
-    </collision>
-    <!-- Define visualization structure -->
-    <visual name='base_link_visual'>
-	  <origin xyz="0 0 0" rpy=" 0 0 0"/>
-      <geometry>
-        <box size="${x_chassis} ${y_chassis} ${z_chassis}"/>
-      </geometry>
-    </visual>
-    <!-- Add the caster wheel! Here we simply assume complete slippage, thus we do not require that it rotates! -->
-    <!-- <collision name='caster_collision'>
-      <origin xyz="${-(r_wheel/2)+x_chassis/2} 0 ${-z_chassis/2}" rpy=" 0 0 0"/>
-      <geometry>
-        <sphere radius="${r_wheel/2}"/>
-      </geometry>
-      <surface>
-        <friction>
-          <ode>
-            <mu>0</mu>
-            <mu2>0</mu2>
-            <slip1>1.0</slip1>
-            <slip2>1.0</slip2>
-          </ode>
-        </friction>
-      </surface>
-    </collision>
-    <visual name='caster_visual'>
-      <origin xyz="${-(r_wheel/2)+x_chassis/2} 0 ${-z_chassis/2}" rpy=" 0 0 0"/>
-      <geometry>
-        <sphere radius="${r_wheel/2}"/>
-      </geometry>
-    </visual> -->
-  </link>
-  <!-- Test Leg -->
-  <link name="leg_rl">
-    <inertial>
-      <mass value="${m_leg}"/>
-      <xacro:box_inertia m="${m_leg}" x="${l_leg}" y="${w_leg}" z="${h_leg}"/>
-    </inertial>
-    <collision name="collision">
-      <origin xyz="0 0 0" rpy="0 0 1.5707"/>
-      <geometry>
-        <box size="${l_leg} ${w_leg} ${h_leg}"/>
-      </geometry>
-    </collision>
-    <visual name="leg_rl_visual">
-      <origin xyz="0 0 0" rpy="0 0 1.5707"/>
-      <geometry>
-        <box size="${l_leg} ${w_leg} ${h_leg}"/>
-      </geometry>
-    </visual>
-  </link>
-  <link name="leg_rr">
-    <inertial>
-      <mass value="${m_leg}"/>
-      <xacro:box_inertia m="${m_leg}" x="${l_leg}" y="${w_leg}" z="${h_leg}"/>
-    </inertial>
-    <collision name="collision">
-      <origin xyz="0 0 0" rpy="0 0 1.5707"/>
-      <geometry>
-        <box size="${l_leg} ${w_leg} ${h_leg}"/>
-      </geometry>
-    </collision>
-    <visual name="leg_rr_visual">
-      <origin xyz="0 0 0" rpy="0 0 1.5707"/>
-      <geometry>
-        <box size="${l_leg} ${w_leg} ${h_leg}"/>
-      </geometry>
-    </visual>
-  </link>
-  <link name="leg_fl">
-    <inertial>
-      <mass value="${m_leg}"/>
-      <xacro:box_inertia m="${m_leg}" x="${l_leg}" y="${w_leg}" z="${h_leg}"/>
-    </inertial>
-    <collision name="collision">
-      <origin xyz="0 0 0" rpy="0 0 1.5707"/>
-      <geometry>
-        <box size="${l_leg} ${w_leg} ${h_leg}"/>
-      </geometry>
-    </collision>
-    <visual name="leg_fl_visual">
-      <origin xyz="0 0 0" rpy="0 0 1.5707"/>
-      <geometry>
-        <box size="${l_leg} ${w_leg} ${h_leg}"/>
-      </geometry>
-    </visual>
-  </link>
-  <link name="leg_fr">
-    <inertial>
-      <mass value="${m_leg}"/>
-      <xacro:box_inertia m="${m_leg}" x="${l_leg}" y="${w_leg}" z="${h_leg}"/>
-    </inertial>
-    <collision name="collision">
-      <origin xyz="0 0 0" rpy="0 0 1.5707"/>
-      <geometry>
-        <box size="${l_leg} ${w_leg} ${h_leg}"/>
-      </geometry>
-    </collision>
-    <visual name="leg_fr_visual">
-      <origin xyz="0 0 0" rpy="0 0 1.5707"/>
-      <geometry>
-        <box size="${l_leg} ${w_leg} ${h_leg}"/>
-      </geometry>
-    </visual>
-  </link>
-  <!-- Add the wheels for the robot -->
-  <link name="wheel_rl">
-    <collision name="collision">
-      <origin xyz="0 0 0" rpy="0 1.5707 1.5707"/>
-      <geometry>
-        <cylinder radius="${r_wheel}" length="${h_wheel}"/>
-      </geometry>
-      <surface>
-        <friction>
-          <ode>
-            <mu>1.0</mu>
-            <mu2>1.0</mu2>
-            <slip1>0.0</slip1>
-            <slip2>0.0</slip2>
-          </ode>
-        </friction>
-      </surface>
-    </collision>
-    <visual name="wheel_rl_visual">
-      <origin xyz="0 0 0" rpy="0 1.5707 1.5707"/>
-      <geometry>
-        <cylinder radius="${r_wheel}" length="${h_wheel}"/>
-      </geometry>
-    </visual>
-    <inertial>
-      <origin xyz="0 0 0" rpy="0 1.5707 1.5707"/>
-      <mass value="${m_wheel}"/>
-      <cylinder_inertia m="${m_wheel}" r="${r_wheel}" h="${h_wheel}"/>
-      <xacro:cylinder_inertia m="${m_wheel}" r="${r_wheel}" h="${h_wheel}"/>
-    </inertial>
-  </link>
-  <link name="wheel_rr">
-    <collision name="collision">
-      <origin xyz="0 0 0" rpy="0 1.5707 1.5707"/>
-      <geometry>
-        <cylinder radius="${r_wheel}" length="${h_wheel}"/>
-      </geometry>
-      <surface>
-        <friction>
-          <ode>
-            <mu>1.0</mu>
-            <mu2>1.0</mu2>
-            <slip1>0.0</slip1>
-            <slip2>0.0</slip2>
-          </ode>
-        </friction>
-      </surface>
-    </collision>
-    <visual name="wheel_rr_visual">
-      <origin xyz="0 0 0" rpy="0 1.5707 1.5707"/>
-      <geometry>
-        <cylinder radius="${r_wheel}" length="${h_wheel}"/>
-      </geometry>
-    </visual>
-    <inertial>
-      <origin xyz="0 0 0" rpy="0 1.5707 1.5707"/>
-      <mass value="${m_wheel}"/>
-      <cylinder_inertia m="${m_wheel}" r="${r_wheel}" h="${h_wheel}"/>
-      <xacro:cylinder_inertia m="${m_wheel}" r="${r_wheel}" h="${h_wheel}"/>
-    </inertial>
-  </link>
-  <!--TEST-->
-  <link name="wheel_fr">
-    <collision name="collision">
-      <origin xyz="0 0 0" rpy="0 1.5707 1.5707"/>
-      <geometry>
-        <cylinder radius="${r_wheel}" length="${h_wheel}"/>
-      </geometry>
-      <surface>
-        <friction>
-          <ode>
-            <mu>1.0</mu>
-            <mu2>1.0</mu2>
-            <slip1>0.0</slip1>
-            <slip2>0.0</slip2>
-          </ode>
-        </friction>
-      </surface>
-    </collision>
-    <visual name="wheel_fr_visual">
-      <origin xyz="0 0 0" rpy="0 1.5707 1.5707"/>
-      <geometry>
-        <cylinder radius="${r_wheel}" length="${h_wheel}"/>
-      </geometry>
-    </visual>
-    <inertial>
-      <origin xyz="0 0 0" rpy="0 1.5707 1.5707"/>
-      <mass value="${m_wheel}"/>
-      <cylinder_inertia m="${m_wheel}" r="${r_wheel}" h="${h_wheel}"/>
-      <xacro:cylinder_inertia m="${m_wheel}" r="${r_wheel}" h="${h_wheel}"/>
-    </inertial>
-  </link>
-  <link name="wheel_fl">
-    <collision name="collision">
-      <origin xyz="0 0 0" rpy="0 1.5707 1.5707"/>
-      <geometry>
-        <cylinder radius="${r_wheel}" length="${h_wheel}"/>
-      </geometry>
-      <surface>
-        <friction>
-          <ode>
-            <mu>1.0</mu>
-            <mu2>1.0</mu2>
-            <slip1>0.0</slip1>
-            <slip2>0.0</slip2>
-          </ode>
-        </friction>
-      </surface>
-    </collision>
-    <visual name="wheel_fl_visual">
-      <origin xyz="0 0 0" rpy="0 1.5707 1.5707"/>
-      <geometry>
-        <cylinder radius="${r_wheel}" length="${h_wheel}"/>
-      </geometry>
-    </visual>
-    <inertial>
-      <origin xyz="0 0 0" rpy="0 1.5707 1.5707"/>
-      <mass value="${m_wheel}"/>
-      <cylinder_inertia m="${m_wheel}" r="${r_wheel}" h="${h_wheel}"/>
-      <xacro:cylinder_inertia m="${m_wheel}" r="${r_wheel}" h="${h_wheel}"/>
-    </inertial>
-  </link>
-  <!-- Set joints for the wheels which can be controlled over ROS -->
-  <!-- it is continuous since it is a wheel-->
-  <joint type="continuous" name="leg_fr_joint_wheel_rl">
-    <origin xyz="0 ${l_leg/2+h_wheel/2} ${r_wheel/2-z_chassis/2}" rpy="0 0 0"/>
-    <child link="wheel_rl"/>
-    <parent link="leg_rl"/>
-    <axis xyz="0 1 0" rpy="0 0 0"/>
-    <!-- velocity here is the max allowed velocity not the acutal velocity-->
-    <limit effort="100" velocity="100"/>
-    <joint_properties damping="0.0" friction="0.0"/>
-  </joint>
-  <joint type="continuous" name="leg_rr_joint_wheel_rr">
-    <origin xyz="0 ${-y_chassis/2-h_wheel/2} ${r_wheel/2-z_chassis/2}" rpy="0 0 0"/>
-    <child link="wheel_rr"/>
-    <parent link="leg_rr"/>
-    <axis xyz="0 1 0" rpy="0 0 0"/>
-    <limit effort="100" velocity="100"/>
-    <joint_properties damping="0.0" friction="0.0"/>
-  </joint>
-  <joint type="continuous" name="leg_fr_joint_wheel_fr">
-    <origin xyz="0 ${-l_leg/2-h_wheel/2} ${r_wheel/2-z_chassis/2}" rpy="0 0 0"/>
-    <child link="wheel_fr"/>
-    <parent link="leg_fr"/>
-    <axis xyz="0 1 0" rpy="0 0 0"/>
-    <limit effort="100" velocity="100"/>
-    <joint_properties damping="0.0" friction="0.0"/>
-  </joint>
-  <joint type="continuous" name="leg_fl_joint_wheel_fl">
-    <origin xyz="0 ${l_leg/2+h_wheel/2} ${r_wheel/2-z_chassis/2}" rpy="0 0 0"/>
-    <child link="wheel_fl"/>
-    <parent link="leg_fl"/>
-    <axis xyz="0 1 0" rpy="0 0 0"/>
-    <limit effort="100" velocity="100"/>
-    <joint_properties damping="0.0" friction="0.0"/>
-  </joint>
-   <joint type="revolute" name="chassis_link_joint_leg_rl">
-    <origin xyz="${-wheel_dist_center} ${y_chassis/2+h_wheel/2} ${r_wheel/2-z_chassis/2}" rpy="0 0 0"/>
-    <child link="leg_rl"/>
-    <parent link="chassis_link"/>
-    <axis xyz="0 1 0" rpy="0 0 0"/>
-    <limit effort="100" velocity="100"/>
-    <joint_properties damping="0.0" friction="0.0"/>
-  </joint>
-  <joint type="revolute" name="chassis_link_joint_leg_rr">
-    <origin xyz="${-wheel_dist_center} ${-y_chassis/2-h_wheel/2} ${r_wheel/2-z_chassis/2}" rpy="0 0 0"/>
-    <child link="leg_rr"/>
-    <parent link="chassis_link"/>
-    <axis xyz="0 1 0" rpy="0 0 0"/>
-    <limit effort="100" velocity="100"/>
-    <joint_properties damping="0.0" friction="0.0"/>
-  </joint>
-  <joint type="revolute" name="chassis_link_joint_leg_fl">
-    <origin xyz="${wheel_dist_center} ${y_chassis/2+h_wheel/2} ${r_wheel/2-z_chassis/2}" rpy="0 0 0"/>
-    <child link="leg_fl"/>
-    <parent link="chassis_link"/>
-    <axis xyz="0 1 0" rpy="0 0 0"/>
-    <limit effort="100" velocity="100"/>
-    <joint_properties damping="0.0" friction="0.0"/>
-  </joint>
-  <joint type="revolute" name="chassis_link_joint_leg_fr">
-    <origin xyz="${wheel_dist_center} ${-y_chassis/2-h_wheel/2} ${r_wheel/2-z_chassis/2}" rpy="0 0 0"/>
-    <child link="leg_fr"/>
-    <parent link="chassis_link"/>
-    <axis xyz="0 1 0" rpy="0 0 0"/>
-    <limit effort="100" velocity="100"/>
-    <joint_properties damping="0.0" friction="0.0"/>
-  </joint>
+  <xacro:include filename="$(find sim_world)/models/common_models/common_models.xacro" />
 </robot>

File: ros/src/rover_world/sim_world/models/arm_mode/macros.xacro (robot description, xacro)
@@ -1,17 +1,3 @@
 <?xml version="1.0"?>
 <robot xmlns:xacro="http://www.ros.org/wiki/xacro">
-  <xacro:macro name="box_inertia" params="m x y z">
-      <inertia
-        ixx="${m*(y*y+z*z)/12}" ixy = "0" ixz = "0"
-        iyy="${m*(x*x+z*z)/12}" iyz = "0"
-        izz="${m*(x*x+z*z)/12}"
-      />
-  </xacro:macro>
-  <xacro:macro name="cylinder_inertia" params="m r h">
-    <inertia
-      ixx="${m*(3*r*r+h*h)/12}" ixy = "0" ixz = "0"
-      iyy="${m*(3*r*r+h*h)/12}" iyz = "0"
-      izz="${m*r*r/2}"
-    />
-  </xacro:macro>
 </robot>

File: ros/src/rover_world/sim_world/models/arm_mode/materials.xacro (robot description, xacro)
@@ -1,8 +1,3 @@
 <?xml version="1.0"?>
 <robot xmlns:xacro="http://www.ros.org/wiki/xacro">
-  <!-- Here we define the material color we may want to use -->
-  <!-- R/G/B-->
-  <material name="orange">
-    <color rgba="${255/255} ${108/255} ${10/255} 1.0"/>
-  </material>
 </robot>

File: ros/src/rover_world/sim_world/models/arm_mode/parameter.xacro (robot description, xacro)
@@ -1,24 +1,3 @@
 <?xml version="1.0"?>
 <robot xmlns:xacro="http://www.ros.org/wiki/xacro">
-  <!-- Define parameter for the differential drive robot -->
-  <!-- Parameter for the chassis, size [m] and mass [kg] -->
-  <xacro:property name="x_chassis" value="1.1176" />
-  <xacro:property name="y_chassis" value="0.4064" />
-  <xacro:property name="z_chassis" value="0.127" />
-  <xacro:property name="m_chassis" value="10.0" />
-  <!-- Parameter for the wheels, radius [m], height [m], mass [kg], torque [Nm], wheelbase [m] -->
-  <xacro:property name="r_wheel" value="0.254"/>
-  <xacro:property name="h_wheel" value="0.254" />
-  <xacro:property name="m_wheel" value="3.0" />
-  <xacro:property name="torque_wheel" value="10" />
-  <xacro:property name="L_wheel" value="0.1788" />
-  <xacro:property name="wheel_dist_center" value="0.5588" />
-  <!-- Parameter for the legs, length [m], width [m], height [m], mass [kg]-->
-  <xacro:property name="l_leg" value="0.3048" />
-  <xacro:property name="w_leg" value="0.1270" />
-  <xacro:property name="h_leg" value="0.1143" />
-  <xacro:property name="m_leg" value="2.0" />
-  <!-- Parameter for the antenna, radius [m], length [m] -->
-  <xacro:property name="r_antenna" value="0.0635" />
-  <xacro:property name="l_antenna" value="1.5748" />
 </robot>

Commit message: Update arm_mode.xarco and parameters, added the base arm(arm_j1) onto the chassis and the second arm (arm_j2) at its correct angle and height.

File: ros/src/rover_world/sim_world/models/arm_mode/arm_mode.xacro (robot description, xacro)
@@ -8,3 +8,86 @@
   <xacro:include filename="$(find sim_world)/models/arm_mode/parameter.xacro" />
   <xacro:include filename="$(find sim_world)/models/common_models/common_models.xacro" />
+  <link name="arm_j1">
+    <collision name="collision">
+      <origin xyz="0 0 0" rpy="0 0 0"/>
+      <geometry>
+        <cylinder radius="${j1_r}" length="${j1_l}"/>
+      </geometry>
+    </collision>
+    <visual name="arm_j1_visual">
+      <origin xyz="0 0 0" rpy="0 0 0"/>
+      <geometry>
+        <cylinder radius="${j1_r}" length="${j1_l}"/>
+      </geometry>
+    </visual>
+    <inertial>
+      <origin xyz="0 0 0" rpy="0 0 0"/>
+      <mass value="1"/>
+      <inertia
+          ixx="1.0" ixy="0.0" ixz="0.0"
+          iyy="1.0" iyz="0.0"
+          izz="1.0"/>
+    </inertial>
+  </link>
+  <link name="arm_j2">
+    <collision name="collision">
+      <origin xyz="0 0 0" rpy="0 0 0"/>
+      <geometry>
+        <cylinder radius="${j2_r}" length="${j2_l}"/>
+      </geometry>
+    </collision>
+    <visual name="arm_j2_visual">
+      <origin xyz="0 0 0" rpy="0 0 0"/>
+      <geometry>
+        <cylinder radius="${j2_r}" length="${j2_l}"/>
+      </geometry>
+    </visual>
+    <inertial>
+      <origin xyz="0 0 0" rpy="0 0 0"/>
+      <mass value="1"/>
+      <inertia
+          ixx="1.0" ixy="0.0" ixz="0.0"
+          iyy="1.0" iyz="0.0"
+          izz="1.0"/>
+    </inertial>
+  </link>
+  <transmission name="j1_tran">
+    <type>transmission_interface/SimpleTransmission</type>
+    <joint name="arm_j1">
+      <hardwareInterface>EffortJointInterface</hardwareInterface>
+    </joint>
+    <actuator name="j1_motor">
+      <hardwareInterface>EffortJointInterface</hardwareInterface>
+      <mechanicalReduction>1</mechanicalReduction>
+    </actuator>
+  </transmission>
+  <transmission name="j2_tran">
+    <type>transmission_interface/SimpleTransmission</type>
+    <joint name="arm_j2">
+      <hardwareInterface>EffortJointInterface</hardwareInterface>
+    </joint>
+    <actuator name="j2_motor">
+      <hardwareInterface>EffortJointInterface</hardwareInterface>
+      <mechanicalReduction>1</mechanicalReduction>
+    </actuator>
+  </transmission>
+  <!-- Joints -->
+  <joint type="revolute" name="chassis_link_arm_j1">
+    <origin xyz="0 0 ${z_chassis/2+j1_l/2}" rpy="0 0 0"/>
+    <child link="arm_j1"/>
+    <parent link="chassis_link"/>
+    <axis xyz="0 1 0" rpy="0 0 0"/>
+    <!-- velocity here is the max allowed velocity not the acutal velocity-->
+    <limit effort="100" velocity="100"/>
+    <joint_properties damping="0.0" friction="0.0"/>
+  </joint>
+    <joint type="revolute" name="arm_j1_arm_j2">
+    <origin xyz="0.2318 0 ${j1_l/2+j2_l/2+0.066802}" rpy="0 1.0887 0"/>
+    <child link="arm_j2"/>
+    <parent link="arm_j1"/>
+    <axis xyz="0 1 0" rpy="0 0 0"/>
+    <!-- velocity here is the max allowed velocity not the acutal velocity-->
+    <limit effort="100" velocity="100"/>
+    <joint_properties damping="0.0" friction="0.0"/>
+  </joint>
 </robot>

File: ros/src/rover_world/sim_world/models/arm_mode/parameter.xacro (robot description, xacro)
@@ -1,3 +1,9 @@
 <?xml version="1.0"?>
 <robot xmlns:xacro="http://www.ros.org/wiki/xacro">
+  <!-- Parameters for arm_21, radius [m] and lenght [m] -->
+    <xacro:property name="j1_r" value="0.124968" />
+    <xacro:property name="j1_l" value="0.040132" />
+  <!-- Parameters for arm_j2, radius [m] and lenght -->
+  <xacro:property name="j2_r" value="0.1016" />
+  <xacro:property name="j2_l" value="0.767842" />
 </robot>
