Commit message: Edited the arm mode with the links and angles up to J5, still need to add the fingers to J5.

File: ros/src/rover_world/sim_world/models/arm_mode/arm_mode.xacro (robot description, xacro)
@@ -32,5 +32,5 @@
   <link name="arm_j2">
     <collision name="collision">
-      <origin xyz="0 0 0" rpy="0 0 0"/>
+      <origin xyz="0 0 ${j2_l/2+0.033401}" rpy="0 0 0"/>
       <geometry>
         <cylinder radius="${j2_r}" length="${j2_l}"/>
@@ -38,5 +38,5 @@
     </collision>
     <visual name="arm_j2_visual">
-      <origin xyz="0 0 0" rpy="0 0 0"/>
+      <origin xyz="0 0 ${j2_l/2+0.033401}" rpy="0 0 0"/>
       <geometry>
         <cylinder radius="${j2_r}" length="${j2_l}"/>
@@ -52,4 +52,70 @@
     </inertial>
   </link>
+  <link name="arm_j3">
+    <collision name="collision">
+      <origin xyz="0 0 ${j3_l/2+0.057}" rpy="0 0 0"/>
+      <geometry>
+        <cylinder radius="${j3_r}" length="${j3_l}"/>
+      </geometry>
+    </collision>
+    <visual name="arm_j3_visual">
+      <origin xyz="0 0 ${j3_l/2+0.057}" rpy="0 0 0"/>
+      <geometry>
+        <cylinder radius="${j3_r}" length="${j3_l}"/>
+      </geometry>
+    </visual>
+    <inertial>
+      <origin xyz="0 0 0" rpy="0 0 0"/>
+      <mass value="1"/>
+      <inertia
+          ixx="1.0" ixy="0.0" ixz="0.0"
+          iyy="1.0" iyz="0.0"
+          izz="1.0"/>
+    </inertial>
+  </link>
+  <link name="arm_j4">
+    <collision name="collision">
+      <origin xyz="0 0 ${j4_l/2+0.07}" rpy="0 0 0"/>
+      <geometry>
+        <cylinder radius="${j4_r}" length="${j4_l}"/>
+      </geometry>
+    </collision>
+    <visual name="arm_j4_visual">
+      <origin xyz="0 0 ${j4_l/2+0.07}" rpy="0 0 0"/>
+      <geometry>
+        <cylinder radius="${j4_r}" length="${j4_l}"/>
+      </geometry>
+    </visual>
+    <inertial>
+      <origin xyz="0 0 0" rpy="0 0 0"/>
+      <mass value="1"/>
+      <inertia
+          ixx="1.0" ixy="0.0" ixz="0.0"
+          iyy="1.0" iyz="0.0"
+          izz="1.0"/>
+    </inertial>
+  </link>
+  <link name="arm_j5">
+    <collision name="collision">
+      <origin xyz="0 0 0" rpy="0 0 0"/>
+      <geometry>
+        <cylinder radius="${j5_r}" length="${j5_l}"/>
+      </geometry>
+    </collision>
+    <visual name="arm_j5_visual">
+      <origin xyz="0 0 0" rpy="0 0 0"/>
+      <geometry>
+        <cylinder radius="${j5_r}" length="${j5_l}"/>
+      </geometry>
+    </visual>
+    <inertial>
+      <origin xyz="0 0 0" rpy="0 0 0"/>
+      <mass value="1"/>
+      <inertia
+          ixx="1.0" ixy="0.0" ixz="0.0"
+          iyy="1.0" iyz="0.0"
+          izz="1.0"/>
+    </inertial>
+  </link>
   <transmission name="j1_tran">
     <type>transmission_interface/SimpleTransmission</type>
@@ -68,4 +134,24 @@
     </joint>
     <actuator name="j2_motor">
+      <hardwareInterface>EffortJointInterface</hardwareInterface>
+      <mechanicalReduction>1</mechanicalReduction>
+    </actuator>
+  </transmission>
+  <transmission name="j3_tran">
+    <type>transmission_interface/SimpleTransmission</type>
+    <joint name="arm_j3">
+      <hardwareInterface>EffortJointInterface</hardwareInterface>
+    </joint>
+    <actuator name="j3_motor">
+      <hardwareInterface>EffortJointInterface</hardwareInterface>
+      <mechanicalReduction>1</mechanicalReduction>
+    </actuator>
+  </transmission>
+  <transmission name="j4_tran">
+    <type>transmission_interface/SimpleTransmission</type>
+    <joint name="arm_j4">
+      <hardwareInterface>EffortJointInterface</hardwareInterface>
+    </joint>
+    <actuator name="j4_motor">
       <hardwareInterface>EffortJointInterface</hardwareInterface>
       <mechanicalReduction>1</mechanicalReduction>
@@ -74,5 +160,5 @@
   <!-- Joints -->
   <joint type="revolute" name="chassis_link_arm_j1">
-    <origin xyz="0 0 ${z_chassis/2+j1_l/2}" rpy="0 0 0"/>
+    <origin xyz="${x_chassis/2-0.62} ${-y_chassis/2+0.207} ${z_chassis/2+j1_l/2}" rpy="0 0 0"/>
     <child link="arm_j1"/>
     <parent link="chassis_link"/>
@@ -82,6 +168,6 @@
     <joint_properties damping="0.0" friction="0.0"/>
   </joint>
-    <joint type="revolute" name="arm_j1_arm_j2">
-    <origin xyz="0.2318 0 ${j1_l/2+j2_l/2+0.066802}" rpy="0 1.0887 0"/>
+  <joint type="revolute" name="arm_j1_arm_j2">
+    <origin xyz="0 0 ${j1_l/2+0.033401}" rpy="0 0.8 0"/>
     <child link="arm_j2"/>
     <parent link="arm_j1"/>
@@ -91,3 +177,30 @@
     <joint_properties damping="0.0" friction="0.0"/>
   </joint>
+  <joint type="revolute" name="arm_j2_arm_j3">
+    <origin xyz="0 0 ${j2_l+0.033401+0.057}" rpy="0 1.0 0"/>
+    <child link="arm_j3"/>
+    <parent link="arm_j2"/>
+    <axis xyz="0 1 0" rpy="0 0 0"/>
+    <!-- velocity here is the max allowed velocity not the acutal velocity-->
+    <limit effort="100" velocity="100"/>
+    <joint_properties damping="0.0" friction="0.0"/>
+  </joint>
+  <joint type="revolute" name="arm_j3_arm_j4">
+    <origin xyz="0 0 ${j3_l+0.057+0.07}" rpy="0 0.7 0"/>
+    <child link="arm_j4"/>
+    <parent link="arm_j3"/>
+    <axis xyz="0 1 0" rpy="0 0 0"/>
+    <!-- velocity here is the max allowed velocity not the acutal velocity-->
+    <limit effort="100" velocity="100"/>
+    <joint_properties damping="0.0" friction="0.0"/>
+  </joint>
+  <joint type="revolute" name="arm_j4_arm_j5">
+    <origin xyz="0 0 ${j4_l+0.07+0.065}" rpy="0 0 0"/>
+    <child link="arm_j5"/>
+    <parent link="arm_j4"/>
+    <axis xyz="0 1 0" rpy="0 0 0"/>
+    <!-- velocity here is the max allowed velocity not the acutal velocity-->
+    <limit effort="100" velocity="100"/>
+    <joint_properties damping="0.0" friction="0.0"/>
+  </joint>
 </robot>

File: ros/src/rover_world/sim_world/models/arm_mode/parameter.xacro (robot description, xacro)
@@ -7,3 +7,12 @@
   <xacro:property name="j2_r" value="0.1016" />
   <xacro:property name="j2_l" value="0.767842" />
+  <!-- Parameters for arm_j3, radius [m] and lenght -->
+  <xacro:property name="j3_r" value="0.1016" />
+  <xacro:property name="j3_l" value="0.435864" />
+  <!-- Parameters for arm_j4, radius [m] and lenght -->
+  <xacro:property name="j4_r" value="0.1016" />
+  <xacro:property name="j4_l" value="0.17145" />
+  <!-- Parameters for arm_j5, radius [m] and lenght -->
+  <xacro:property name="j5_r" value="0.1016" />
+  <xacro:property name="j5_l" value="0.122936" />
 </robot>

Commit message: Working on the meshes, edited the common and arm xarcos as well as adding meshes to the mesh folder

File: ros/src/rover_world/sim_world/models/arm_mode/arm_mode.xacro (robot description, xacro)
@@ -18,5 +18,6 @@
       <origin xyz="0 0 0" rpy="0 0 0"/>
       <geometry>
-        <cylinder radius="${j1_r}" length="${j1_l}"/>
+        <mesh filename="package://sim_world/meshes/J1v2.dae"/>
+        <!-- <cylinder radius="${j1_r}" length="${j1_l}"/> -->
       </geometry>
     </visual>
@@ -40,5 +41,6 @@
       <origin xyz="0 0 ${j2_l/2+0.033401}" rpy="0 0 0"/>
       <geometry>
-        <cylinder radius="${j2_r}" length="${j2_l}"/>
+        <mesh filename="package://sim_world/meshes/J2 fixedv2.dae"/>
+        <!-- <cylinder radius="${j2_r}" length="${j2_l}"/> -->
       </geometry>
     </visual>
@@ -62,5 +64,6 @@
       <origin xyz="0 0 ${j3_l/2+0.057}" rpy="0 0 0"/>
       <geometry>
-        <cylinder radius="${j3_r}" length="${j3_l}"/>
+        <mesh filename="package://sim_world/meshes/J3v2.dae"/>
+        <!-- <cylinder radius="${j3_r}" length="${j3_l}"/> -->
       </geometry>
     </visual>
@@ -84,5 +87,6 @@
       <origin xyz="0 0 ${j4_l/2+0.07}" rpy="0 0 0"/>
       <geometry>
-        <cylinder radius="${j4_r}" length="${j4_l}"/>
+        <mesh filename="package://sim_world/meshes/J4redov2.dae"/>
+        <!-- <cylinder radius="${j4_r}" length="${j4_l}"/> -->
       </geometry>
     </visual>
@@ -106,5 +110,6 @@
       <origin xyz="0 0 0" rpy="0 0 0"/>
       <geometry>
-        <cylinder radius="${j5_r}" length="${j5_l}"/>
+        <mesh filename="package://sim_world/meshes/J5.dae"/>
+        <!-- <cylinder radius="${j5_r}" length="${j5_l}"/> -->
       </geometry>
     </visual>

File: ros/src/rover_world/sim_world/models/common_models/common_models.xacro (robot description, xacro)
@@ -34,5 +34,6 @@
 	  <origin xyz="0 0 0" rpy=" 0 0 0"/>
       <geometry>
-        <box size="${x_chassis} ${y_chassis} ${z_chassis}"/>
+        <mesh filename="package://sim_world/meshes/chassis-w-baseplate.dae"/>
+        <!-- <box size="${x_chassis} ${y_chassis} ${z_chassis}"/> -->
       </geometry>
     </visual>
@@ -89,5 +90,6 @@
       <origin xyz="0 0 0" rpy="0 0 ${pi/2}"/>
       <geometry>
-        <box size="${l_leg} ${w_leg} ${h_leg}"/>
+        <mesh filename="package://sim_world/meshes/tr_leg.dae"/>
+        <!-- <box size="${l_leg} ${w_leg} ${h_leg}"/> -->
       </geometry>
     </visual>
@@ -107,5 +109,6 @@
       <origin xyz="0 0 0" rpy="0 0 ${pi/2}"/>
       <geometry>
-        <box size="${l_leg} ${w_leg} ${h_leg}"/>
+        <mesh filename="package://sim_world/meshes/tr_leg.dae"/>
+        <!-- <box size="${l_leg} ${w_leg} ${h_leg}"/> -->
       </geometry>
     </visual>
@@ -125,5 +128,6 @@
       <origin xyz="0 0 0" rpy="0 0 ${pi/2}"/>
       <geometry>
-        <box size="${l_leg} ${w_leg} ${h_leg}"/>
+        <mesh filename="package://sim_world/meshes/Control_armsFL.dae"/>
+        <!-- <box size="${l_leg} ${w_leg} ${h_leg}"/> -->
       </geometry>
     </visual>
@@ -143,5 +147,6 @@
       <origin xyz="0 0 0" rpy="0 0 ${pi/2}"/>
       <geometry>
-        <box size="${l_leg} ${w_leg} ${h_leg}"/>
+        <mesh filename="package://sim_world/meshes/Control_armsFRv2.dae"/>
+        <!-- <box size="${l_leg} ${w_leg} ${h_leg}"/> -->
       </geometry>
     </visual>
@@ -168,5 +173,6 @@
       <origin xyz="0 0 0" rpy="0 ${pi/2} ${pi/2}"/>
       <geometry>
-        <cylinder radius="${r_wheel}" length="${h_wheel}"/>
+        <mesh filename="package://sim_world/meshes/tr_wheel_left.dae"/>
+        <!-- <cylinder radius="${r_wheel}" length="${h_wheel}"/> -->
       </geometry>
     </visual>
@@ -198,5 +204,6 @@
       <origin xyz="0 0 0" rpy="0 ${pi/2} ${pi/2}"/>
       <geometry>
-        <cylinder radius="${r_wheel}" length="${h_wheel}"/>
+        <mesh filename="package://sim_world/meshes/tr_wheel_right.dae"/>
+        <!-- <cylinder radius="${r_wheel}" length="${h_wheel}"/> -->
       </geometry>
     </visual>
@@ -228,5 +235,6 @@
       <origin xyz="0 0 0" rpy="0 ${pi/2} ${pi/2}"/>
       <geometry>
-        <cylinder radius="${r_wheel}" length="${h_wheel}"/>
+        <mesh filename="package://sim_world/meshes/tr_wheel_right.dae"/>
+        <!-- <cylinder radius="${r_wheel}" length="${h_wheel}"/> -->
       </geometry>
     </visual>
@@ -258,5 +266,6 @@
       <origin xyz="0 0 0" rpy="0 ${pi/2} ${pi/2}"/>
       <geometry>
-        <cylinder radius="${r_wheel}" length="${h_wheel}"/>
+        <mesh filename="package://sim_world/meshes/tr_wheel_left.dae"/>
+        <!-- <cylinder radius="${r_wheel}" length="${h_wheel}"/> -->
       </geometry>
     </visual>
